File: PCB-Design/Master Node/MasterNode.brd (EAGLE design)
At the start: 56.6 x 59.6 mm, 9 parts, among them J2 455-1750-1-ND, J4 RJ45

Commit message: New Master Node
Connections:
- net N$5: now also IC1.18; no longer IC1.22
Routing:
- net N$2: track 14.4 -> 47.5 mm
- net N$5: track 76.8 -> 88.8 mm
- net N$1: track 18.3 -> 20.0 mm
Other:
- board size 56.6 x 59.6 mm -> 54.3 x 59.6 mm
